Commit message: load objects

File: objects_model/objs/meshes/2c0600cdf28535eb8dfc720b465c725c.urdf (robot description, URDF)
Before this commit: robot cube.urdf, 1 links, 0 joints
Links:
- link legobrick: geometry collision mesh filename=2c0600cdf28535eb8dfc720b465c725c_col.obj scale=1.2 1.2 1.2; visual mesh filename=2c0600cdf28535eb8dfc720b465c725c.obj scale=1.2 1.2 1.2

File: objects_model/objs/meshes/2c97e6b2c92913cac1ccec171a275967.urdf (robot description, URDF)
Before this commit: robot cube.urdf, 1 links, 0 joints
Links:
- link legobrick: geometry collision mesh filename=2c97e6b2c92913cac1ccec171a275967_col.obj scale=1.2 1.2 1.2; visual mesh filename=2c97e6b2c92913cac1ccec171a275967.obj scale=1.2 1.2 1.2

File: objects_model/objs/meshes/2c9ec139a84e56dc4f7c5cc287db4b75_1.urdf (robot description, URDF)
Before this commit: robot cube.urdf, 1 links, 0 joints
Links:
- link legobrick: geometry collision mesh filename=2c9ec139a84e56dc4f7c5cc287db4b75_1_col.obj scale=1.2 1.2 1.2; visual mesh filename=2c9ec139a84e56dc4f7c5cc287db4b75_1.obj scale=1.2 1.2 1.2

File: objects_model/objs/meshes/2cad1ab3b30cfc29eb1db99dff281a57.urdf (robot description, URDF)
Before this commit: robot cube.urdf, 1 links, 0 joints
Links:
- link legobrick: geometry collision mesh filename=2cad1ab3b30cfc29eb1db99dff281a57_col.obj scale=1.2 1.2 1.2; visual mesh filename=2cad1ab3b30cfc29eb1db99dff281a57.obj scale=1.2 1.2 1.2

File: objects_model/objs/meshes/2ea71440efc67b9361fc15298b411505.urdf (robot description, URDF)
Before this commit: robot cube.urdf, 1 links, 0 joints
Links:
- link legobrick: geometry collision mesh filename=2ea71440efc67b9361fc15298b411505_col.obj scale=1.2 1.2 1.2; visual mesh filename=2ea71440efc67b9361fc15298b411505.obj scale=1.2 1.2 1.2

File: objects_model/objs/meshes/403fb4eb4fc6235adf0c7dbe7f8f4c8e_1.urdf (robot description, URDF)
Before this commit: robot cube.urdf, 1 links, 0 joints
Links:
- link legobrick: geometry collision mesh filename=403fb4eb4fc6235adf0c7dbe7f8f4c8e_1_col.obj scale=1.2 1.2 1.2; visual mesh filename=403fb4eb4fc6235adf0c7dbe7f8f4c8e_1.obj scale=1.2 1.2 1.2

File: objects_model/objs/meshes/405f308492a6f40d2c3380317c2cc450_1.urdf (robot description, URDF)
Before this commit: robot cube.urdf, 1 links, 0 joints
Links:
- link legobrick: geometry collision mesh filename=405f308492a6f40d2c3380317c2cc450_1_col.obj scale=1.2 1.2 1.2; visual mesh filename=405f308492a6f40d2c3380317c2cc450_1.obj scale=1.2 1.2 1.2

File: objects_model/objs/meshes/407eab234d7c9c4791d13947d0d17396_1.urdf (robot description, URDF)
Before this commit: robot cube.urdf, 1 links, 0 joints
Links:
- link legobrick: geometry collision mesh filename=407eab234d7c9c4791d13947d0d17396_1_col.obj scale=1.2 1.2 1.2; visual mesh filename=407eab234d7c9c4791d13947d0d17396_1.obj scale=1.2 1.2 1.2

File: objects_model/objs/meshes/411b82e61eaf14a8542a0a586afb6486_1.urdf (robot description, URDF)
Before this commit: robot cube.urdf, 1 links, 0 joints
Links:
- link legobrick: geometry collision mesh filename=411b82e61eaf14a8542a0a586afb6486_1_col.obj scale=1.2 1.2 1.2; visual mesh filename=411b82e61eaf14a8542a0a586afb6486_1.obj scale=1.2 1.2 1.2

File: objects_model/objs/meshes/420f6d4f07c3109bee5e7ed304cc3a4c.urdf (robot description, URDF)
Before this commit: robot cube.urdf, 1 links, 0 joints
Links:
- link legobrick: geometry collision mesh filename=420f6d4f07c3109bee5e7ed304cc3a4c_col.obj scale=1.2 1.2 1.2; visual mesh filename=420f6d4f07c3109bee5e7ed304cc3a4c.obj scale=1.2 1.2 1.2

File: objects_model/objs/meshes/48e26e789524c158e1e4b7162e96446c.urdf (robot description, URDF)
Before this commit: robot cube.urdf, 1 links, 0 joints
Links:
- link legobrick: geometry collision mesh filename=48e26e789524c158e1e4b7162e96446c_col.obj scale=1.2 1.2 1.2; visual mesh filename=48e26e789524c158e1e4b7162e96446c.obj scale=1.2 1.2 1.2

File: objects_model/objs/meshes/4b4782c572fa8b11a20c7111a5d0d7fc_1.urdf (robot description, URDF)
Before this commit: robot cube.urdf, 1 links, 0 joints
Links:
- link legobrick: geometry collision mesh filename=4b4782c572fa8b11a20c7111a5d0d7fc_1_col.obj scale=1.2 1.2 1.2; visual mesh filename=4b4782c572fa8b11a20c7111a5d0d7fc_1.obj scale=1.2 1.2 1.2

File: objects_model/objs/meshes/4c5c32eaaf1fc80aa413908c0e169330.urdf (robot description, URDF)
Before this commit: robot cube.urdf, 1 links, 0 joints
Links:
- link legobrick: geometry collision mesh filename=4c5c32eaaf1fc80aa413908c0e169330_col.obj scale=1.2 1.2 1.2; visual mesh filename=4c5c32eaaf1fc80aa413908c0e169330.obj scale=1.2 1.2 1.2

File: objects_model/objs/meshes/4d99955663a6f1d66138f18acdeb955a.urdf (robot description, URDF)
Before this commit: robot cube.urdf, 1 links, 0 joints
Links:
- link legobrick: geometry collision mesh filename=4d99955663a6f1d66138f18acdeb955a_col.obj scale=1.2 1.2 1.2; visual mesh filename=4d99955663a6f1d66138f18acdeb955a.obj scale=1.2 1.2 1.2

File: objects_model/objs/meshes/4dbb5a6cd26d13067964ba700cd97f5.urdf (robot description, URDF)
Before this commit: robot cube.urdf, 1 links, 0 joints
Links:
- link legobrick: geometry collision mesh filename=4dbb5a6cd26d13067964ba700cd97f5_col.obj scale=1.2 1.2 1.2; visual mesh filename=4dbb5a6cd26d13067964ba700cd97f5.obj scale=1.2 1.2 1.2

File: objects_model/objs/meshes/4dc44c77b66c82b9e7f746bc520f60fd.urdf (robot description, URDF)
Before this commit: robot cube.urdf, 1 links, 0 joints
Links:
- link legobrick: geometry collision mesh filename=4dc44c77b66c82b9e7f746bc520f60fd_col.obj scale=1.2 1.2 1.2; visual mesh filename=4dc44c77b66c82b9e7f746bc520f60fd.obj scale=1.2 1.2 1.2

File: objects_model/objs/meshes/57c718fc5c3f79a1203f35d9b3b48203.urdf (robot description, URDF)
Before this commit: robot cube.urdf, 1 links, 0 joints
Links:
- link legobrick: geometry collision mesh filename=57c718fc5c3f79a1203f35d9b3b48203_col.obj scale=1.2 1.2 1.2; visual mesh filename=57c718fc5c3f79a1203f35d9b3b48203.obj scale=1.2 1.2 1.2

File: objects_model/objs/meshes/6e9cdf80e2856c03906d13a17c966645.urdf (robot description, URDF)
Before this commit: robot cube.urdf, 1 links, 0 joints
Links:
- link legobrick: geometry collision mesh filename=6e9cdf80e2856c03906d13a17c966645_col.obj scale=1.2 1.2 1.2; visual mesh filename=6e9cdf80e2856c03906d13a17c966645.obj scale=1.2 1.2 1.2

File: objects_model/objs/meshes/6ed8841f75fe0b87eb5d382c7eb13b28_1.urdf (robot description, URDF)
Before this commit: robot cube.urdf, 1 links, 0 joints
Links:
- link legobrick: geometry collision mesh filename=6ed8841f75fe0b87eb5d382c7eb13b28_1_col.obj scale=1.2 1.2 1.2; visual mesh filename=6ed8841f75fe0b87eb5d382c7eb13b28_1.obj scale=1.2 1.2 1.2

File: objects_model/objs/meshes/6f8062392721742962a30a51f7713338_1.urdf (robot description, URDF)
Before this commit: robot cube.urdf, 1 links, 0 joints
Links:
- link legobrick: geometry collision mesh filename=6f8062392721742962a30a51f7713338_1_col.obj scale=1.2 1.2 1.2; visual mesh filename=6f8062392721742962a30a51f7713338_1.obj scale=1.2 1.2 1.2
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